File: Eagle files/BacKey for MaKey MaKey (rev A).brd (EAGLE design)
At the start: 94 x 38.1 mm, 5 parts

Commit message: Cleaned up schematic a bit
Parts:
- removed JP14: (no value), SparkFun-Connectors:1X06
- added JP4: (no value), SparkFun-Connectors:1X06
- moved JP1 84.8 mm to (5.08, 13.5), turned to 90 degrees
- moved JP2 43.2 mm to (43.2, 33.8), turned to 180 degrees
- moved JP3 42.3 mm to (88.9, 26.2), turned to 270 degrees
Connections:
- net A0: now also JP1.1; no longer JP2.1
- net A1: now also JP1.2; no longer JP2.2
- net A2: now also JP1.3; no longer JP2.3
- net A3: now also JP1.4; no longer JP2.4
- net A4: now also JP1.5; no longer JP2.5
- net A5: now also JP1.6; no longer JP2.6
- net D0: now also JP3.6; no longer JP1.6
- net D1: now also JP3.5; no longer JP1.5
- net D14: now also JP2.6; no longer JP14.6
- net D15: now also JP2.1; no longer JP14.1
- net D16: now also JP2.5; no longer JP14.5
- net D2: now also JP3.4; no longer JP1.4
- net D3: now also JP3.3; no longer JP1.3
- net D4: now also JP3.2; no longer JP1.2
- net D5: now also JP3.1; no longer JP1.1
- net GND: now also JP2.3, JP4.1, JP4.2, JP4.3, JP4.4, JP4.5, JP4.6; no longer JP14.3, JP3.1, JP3.2, JP3.3, JP3.4, JP3.5, JP3.6
- net RESET: now also JP2.2; no longer JP14.2
- net VCC: now also JP2.4; no longer JP14.4
Changed lines of the file:
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@@
 <elements>
 <element name="U$1" library="SparkFun-Aesthetics" package="OSHW-LOGO-M" value="OSHW-LOGOM" x="80.137" y="33.147" rot="MR0"/>
-<element name="JP3" library="SparkFun-Connectors" package="1X06" value="" x="53.34" y="3.302" smashed="yes" rot="MR0">
+<element name="JP4" library="SparkFun-Connectors" package="1X06" value="" x="53.34" y="3.302" smashed="yes" rot="MR0">
 <attribute name="VALUE" x="54.61" y="0.127" size="1.27" layer="28" rot="MR0"/>
 </element>
-<element name="JP14" library="SparkFun-Connectors" package="1X06" value="" x="43.18" y="33.782" smashed="yes" rot="MR180">
+<element name="JP2" library="SparkFun-Connectors" package="1X06" value="" x="43.18" y="33.782" smashed="yes" rot="MR180">
 <attribute name="VALUE" x="41.91" y="36.957" size="1.27" layer="28" rot="MR180"/>
 </element>
-<element name="JP1" library="SparkFun-Connectors" package="1X06" value="" x="88.9" y="26.162" smashed="yes" rot="MR270">
+<element name="JP3" library="SparkFun-Connectors" package="1X06" value="" x="88.9" y="26.162" smashed="yes" rot="MR270">
 <attribute name="VALUE" x="92.075" y="27.432" size="1.27" layer="28" rot="MR270"/>
 </element>
-<element name="JP2" library="SparkFun-Connectors" package="1X06" value="" x="5.08" y="13.462" smashed="yes" rot="MR90">
+<element name="JP1" library="SparkFun-Connectors" package="1X06" value="" x="5.08" y="13.462" smashed="yes" rot="MR90">
 <attribute name="VALUE" x="1.905" y="12.192" size="1.27" layer="28" rot="MR90"/>
 </element>
@@
 <vertex x="89.027" y="38.1"/>
 </polygon>
-<contactref element="JP3" pad="1"/>
-<contactref element="JP3" pad="2"/>
-<contactref element="JP3" pad="3"/>
-<contactref element="JP3" pad="4"/>
-<contactref element="JP3" pad="5"/>
-<contactref element="JP3" pad="6"/>
-<contactref element="JP14" pad="3"/>
+<contactref element="JP4" pad="1"/>
+<contactref element="JP4" pad="2"/>
+<contactref element="JP4" pad="3"/>
+<contactref element="JP4" pad="4"/>
+<contactref element="JP4" pad="5"/>
+<contactref element="JP4" pad="6"/>
+<contactref element="JP2" pad="3"/>
 </signal>
 <signal name="RESET">
-<contactref element="JP14" pad="2"/>
+<contactref element="JP2" pad="2"/>
 </signal>
 <signal name="VCC">
-<contactref element="JP14" pad="4"/>
+<contactref element="JP2" pad="4"/>
 </signal>
 <signal name="D16">
-<contactref element="JP14" pad="5"/>
+<contactref element="JP2" pad="5"/>
 </signal>
 <signal name="D14">
-<contactref element="JP14" pad="6"/>
+<contactref element="JP2" pad="6"/>
 </signal>
 <signal name="D15">
-<contactref element="JP14" pad="1"/>
+<contactref element="JP2" pad="1"/>
 </signal>
 <signal name="A0">
@@
 <via x="22.098" y="10.922" extent="1-16" drill="3.2"/>
 <wire x1="26.67" y1="10.922" x2="22.098" y2="10.922" width="0.6096" layer="16"/>
-<contactref element="JP2" pad="1"/>
+<contactref element="JP1" pad="1"/>
 <wire x1="5.08" y1="13.462" x2="7.62" y2="10.922" width="0.4064" layer="16"/>
 <wire x1="7.62" y1="10.922" x2="22.098" y2="10.922" width="0.4064" layer="16"/>
@@
 <via x="34.798" y="10.922" extent="1-16" drill="3.2"/>
 <wire x1="39.37" y1="10.922" x2="34.798" y2="10.922" width="0.6096" layer="16"/>
-<contactref element="JP2" pad="2"/>
+<contactref element="JP1" pad="2"/>
 <wire x1="5.08" y1="16.002" x2="6.858" y2="14.224" width="0.4064" layer="16"/>
 <wire x1="6.858" y1="14.224" x2="31.496" y2="14.224" width="0.4064" layer="16"/>
@@
 <via x="22.098" y="17.272" extent="1-16" drill="3.2"/>
 <wire x1="26.67" y1="17.272" x2="22.098" y2="17.272" width="0.6096" layer="16"/>
-<contactref element="JP2" pad="3"/>
+<contactref element="JP1" pad="3"/>
 <wire x1="5.08" y1="18.542" x2="20.828" y2="18.542" width="0.4064" layer="16"/>
 <wire x1="20.828" y1="18.542" x2="22.098" y2="17.272" width="0.4064" layer="16"/>
@@
 <wire x1="34.798" y1="17.526" x2="34.798" y2="17.272" width="0.6096" layer="16"/>
 <wire x1="39.37" y1="17.272" x2="35.306" y2="17.272" width="0.6096" layer="16"/>
-<contactref element="JP2" pad="4"/>
+<contactref element="JP1" pad="4"/>
 <wire x1="35.306" y1="17.272" x2="34.798" y2="17.272" width="0.6096" layer="16"/>
 <wire x1="5.08" y1="21.082" x2="6.096" y2="20.574" width="0.4064" layer="16"/>
@@
 <via x="22.098" y="23.622" extent="1-16" drill="3.2"/>
 <wire x1="26.67" y1="23.622" x2="22.098" y2="23.622" width="0.6096" layer="16"/>
-<contactref element="JP2" pad="5"/>
+<contactref element="JP1" pad="5"/>
 <wire x1="5.08" y1="23.622" x2="22.098" y2="23.622" width="0.4064" layer="16"/>
 </signal>
@@
 <via x="34.798" y="23.622" extent="1-16" drill="3.2"/>
 <wire x1="39.37" y1="23.622" x2="34.798" y2="23.622" width="0.6096" layer="16"/>
-<contactref element="JP2" pad="6"/>
+<contactref element="JP1" pad="6"/>
 <wire x1="5.08" y1="26.162" x2="6.096" y2="27.178" width="0.4064" layer="16"/>
 <wire x1="6.096" y1="27.178" x2="32.004" y2="27.178" width="0.4064" layer="16"/>
@@
 <via x="70.358" y="10.922" extent="1-16" drill="3.2"/>
 <wire x1="70.358" y1="10.922" x2="74.93" y2="10.922" width="0.6096" layer="16"/>
-<contactref element="JP1" pad="6"/>
+<contactref element="JP3" pad="6"/>
 <wire x1="88.9" y1="13.462" x2="86.36" y2="10.922" width="0.4064" layer="16"/>
 <wire x1="86.36" y1="10.922" x2="74.93" y2="10.922" width="0.4064" layer="16"/>
@@
 <wire x1="62.738" y1="10.922" x2="62.23" y2="10.922" width="0.6096" layer="16"/>
 <wire x1="57.658" y1="10.922" x2="62.23" y2="10.922" width="0.6096" layer="16"/>
-<contactref element="JP1" pad="5"/>
+<contactref element="JP3" pad="5"/>
 <wire x1="88.9" y1="16.002" x2="87.122" y2="14.224" width="0.4064" layer="16"/>
 <wire x1="87.122" y1="14.224" x2="66.04" y2="14.224" width="0.4064" layer="16"/>
@@
 <via x="70.358" y="17.272" extent="1-16" drill="3.2"/>
 <wire x1="70.358" y1="17.272" x2="74.93" y2="17.272" width="0.6096" layer="16"/>
-<contactref element="JP1" pad="4"/>
+<contactref element="JP3" pad="4"/>
 <wire x1="88.9" y1="18.542" x2="76.2" y2="18.542" width="0.4064" layer="16"/>
 <wire x1="76.2" y1="18.542" x2="74.93" y2="17.272" width="0.4064" layer="16"/>
@@
 <wire x1="63.246" y1="17.272" x2="62.23" y2="17.272" width="0.6096" layer="16"/>
 <wire x1="57.658" y1="17.272" x2="62.23" y2="17.272" width="0.6096" layer="16"/>
-<contactref element="JP1" pad="3"/>
+<contactref element="JP3" pad="3"/>
 <wire x1="88.9" y1="21.082" x2="88.138" y2="20.32" width="0.4064" layer="16"/>
 <wire x1="88.138" y1="20.32" x2="66.294" y2="20.32" width="0.4064" layer="16"/>
@@
 <via x="70.358" y="23.622" extent="1-16" drill="3.2"/>
 <wire x1="70.358" y1="23.622" x2="74.93" y2="23.622" width="0.6096" layer="16"/>
-<contactref element="JP1" pad="2"/>
+<contactref element="JP3" pad="2"/>
 <wire x1="88.9" y1="23.622" x2="74.93" y2="23.622" width="0.4064" layer="16"/>
 </signal>
@@
 <wire x1="62.738" y1="23.622" x2="62.23" y2="23.622" width="0.6096" layer="16"/>
 <wire x1="57.658" y1="23.622" x2="62.23" y2="23.622" width="0.6096" layer="16"/>
-<contactref element="JP1" pad="1"/>
+<contactref element="JP3" pad="1"/>
 <wire x1="62.738" y1="23.622" x2="66.04" y2="26.924" width="0.4064" layer="16"/>
 <wire x1="66.04" y1="26.924" x2="88.392" y2="26.924" width="0.4064" layer="16"/>
